Commit message: Port emma's base driving and display lessons to the template
Add a pixi display task and an initial argument on the position_joint
macro, with a note to keep starting poses strictly inside joint limits.

Document what emma's mecanum base needed: wheel joints with velocity
interfaces, motor actuators with a PID file, wheel armature, roller
post-processing, per-controller TF remaps, a sim RViz config rooted at
odom, and a physics-only drive check.

File: src/my_robot_description/urdf/my_robot.urdf.xacro (robot description, xacro)
@@ -69,9 +69,11 @@
   <xacro:arg name="mujoco_model" default=""/>
   <xacro:arg name="headless" default="false"/>
-  <xacro:macro name="position_joint" params="name">
+  <!-- initial is the joint position MuJoCo starts at. Keep it strictly inside the joint
+       limits: exactly on a limit, numerical drift trips the joint limiter. -->
+  <xacro:macro name="position_joint" params="name initial:=0.0">
     <joint name="${name}">
       <command_interface name="position"/>
       <state_interface name="position">
-        <param name="initial_value">0.0</param>
+        <param name="initial_value">${initial}</param>
       </state_interface>
       <state_interface name="velocity"/>
